File: Proyecto4.kicad_pcb (KiCad board)
At the start: 4 copper layers, 42 x 42 mm, 111 parts, among them J1 Conn_01x05_Female, J2 USB_C_Receptacle_USB2.0, J4 PV Panel 1, J5 PV Panel 2, J6 Battery, J7 Conn_02x20_Odd_Even, J8 Conn_02x20_Odd_Even, Q1 SQ3989EV, Q2 DMG2305, SW1 SW_Push, SW2 SW_SPDT, U1 ATSAMD21G18A, U10 TPS22918, U11 TPS22918, U2 GD25Q32, U3 INA226, U4 FP6291, U5 TPS22918, U6 SPV1040, U7 SY8089, U8 L6924D, U9 TPS22918, Y1 32.768 kHz - 12.5pF

Commit message: Final
Parts:
- removed C10, C12, C26: 10nF, Capacitor_SMD:C_0402_1005Metric
- removed C11, C18, C25, C27: 1uF, Capacitor_SMD:C_0402_1005Metric
- removed C13, C30: 10uF, Capacitor_SMD:C_0603_1608Metric
- removed C14, C19, C23, C29: 100nF, Capacitor_SMD:C_0402_1005Metric
- removed C15, C16, C20, C22, C24: 22uF, Capacitor_SMD:C_0603_1608Metric
- removed C17: 1nF, Capacitor_SMD:C_0402_1005Metric
- removed C21: 4.7F, Capacitor_SMD:C_0603_1608Metric
- removed C28: 1uF, Capacitor_SMD:C_0603_1608Metric
- removed C31, C32: 220uF, Capacitor_SMD:C_1206_3216Metric
- removed D1: WS2812B, DynOSSAT:LED_SK6812MINI_PLCC4_3.5x3.5mm_P1.75mm
- removed D10, D5, D7, D8, D9: D_Schottky_Small, Diode_SMD:D_SOD-323
- removed D6: D_Schottky_Small, Diode_SMD:D_SOD-123
- removed G***: LOGO, DynOSSAT:Logo_BHDyn
- removed the J2 at (194.8, 82.2)
- removed J6: Battery, DynOSSAT:Molex_PicoBlade_53048-0210_1x02_P1.25mm_Horizontal
- removed the J7 at (208.6, 52.6)
- removed JP1: Jumper, Connector_PinHeader_1.27mm:PinHeader_1x02_P1.27mm_Vertical
- removed JP2: Jumper, Jumper:SolderJumper-2_P1.3mm_Bridged_RoundedPad1.0x1.5mm
- removed L3: 3.3uH, Inductor_SMD:L_1210_3225Metric
- removed Q1: SQ3989EV, Package_TO_SOT_SMD:SOT-23-6
- removed Q2: DMG2305, Package_TO_SOT_SMD:SOT-23
- removed R10, R25: 1M, Resistor_SMD:R_0402_1005Metric
- removed R11, R18, R27, R32: 100k, Resistor_SMD:R_0402_1005Metric
- removed R12, R13: 330R, Resistor_SMD:R_0402_1005Metric
- removed R14, R15, R16: 1k, Resistor_SMD:R_0402_1005Metric
- removed R17: 0.033R, Resistor_SMD:R_0603_1608Metric
- removed R19: 22k2, Resistor_SMD:R_0402_1005Metric
- removed R20: 2.2M, Resistor_SMD:R_0402_1005Metric
- removed R21: 820k, Resistor_SMD:R_0402_1005Metric
- removed R22, R23: 5.1k, Resistor_SMD:R_0402_1005Metric
- removed R24: 10M, Resistor_SMD:R_0402_1005Metric
- removed R26: 1.5M, Resistor_SMD:R_0402_1005Metric
- removed R29, R33, R8, R9: 47k, Resistor_SMD:R_0402_1005Metric
- removed R30: 88k, Resistor_SMD:R_0402_1005Metric
- removed R31, R35: 12k, Resistor_SMD:R_0402_1005Metric
- removed R36: 3k3, Resistor_SMD:R_0402_1005Metric
- removed R7: 0.002R, Resistor_SMD:R_0603_1608Metric
- removed the REF** at (217.7, 85.5)
- removed SW1: SW_Push, DynOSSAT:1TS002G-1800-3500-CT
- removed U10, U11, U5, U9: TPS22918, Package_TO_SOT_SMD:SOT-23-6
- removed U2: GD25Q32, DynOSSAT:WSON-8-1EP_3x4mm_P0.8mm
- removed U4: FP6291, Package_TO_SOT_SMD:SOT-23-6
- removed U6: SPV1040, Package_SO:TSSOP-8_4.4x3mm_P0.65mm
- removed U7: SY8089, Package_TO_SOT_SMD:SOT-23-5
- removed U8: L6924D, DynOSSAT:VQFN-16-1EP_3x3mm_P0.5mm_EP1.45x1.45mm
- removed Y1: 32.768 kHz - 12.5pF, DynOSSAT:Crystal_SMD_2012-2Pin_2.0x1.2mm
- added J1: Conn_02x20_Odd_Even, Connector_PinHeader_1.27mm:PinHeader_2x20_P1.27mm_Vertical_SMD, F.Cu at (208.6, 52.6)
- added J3: Battery, DynOSSAT:Molex_PicoBlade_53048-0210_1x02_P1.25mm_Horizontal, F.Cu at (192.8, 59.9)
- C1: value 22pF -> 4.9uF; footprint Capacitor_SMD:C_0402_1005Metric -> Capacitor_SMD:C_0603_1608Metric
- C2: value 22pF -> 4.7uF; footprint Capacitor_SMD:C_0402_1005Metric -> Capacitor_SMD:C_0603_1608Metric
- C3: value 1nF -> 470nF; footprint Capacitor_SMD:C_0402_1005Metric -> Capacitor_SMD:C_0603_1608Metric
- C4: value 100nF -> 4.9uF; footprint Capacitor_SMD:C_0402_1005Metric -> Capacitor_SMD:C_0603_1608Metric
- C5: value 100nF -> 1.01uF; footprint Capacitor_SMD:C_0402_1005Metric -> Capacitor_SMD:C_0603_1608Metric
- C6: value 100nF -> 4.7uF; footprint Capacitor_SMD:C_0402_1005Metric -> Capacitor_SMD:C_0603_1608Metric
- C7: value 100nF -> 3.3nF; footprint Capacitor_SMD:C_0402_1005Metric -> Capacitor_SMD:C_0603_1608Metric
- C8: value 100nF -> 0.1uF; footprint Capacitor_SMD:C_0402_1005Metric -> Capacitor_SMD:C_0603_1608Metric
- C9: value 100nF -> 10uF; footprint Capacitor_SMD:C_0402_1005Metric -> Capacitor_SMD:C_Elec_4x5.4
- D3: value LED_Small -> D_Schottky_Small; footprint LED_SMD:LED_0603_1608Metric -> Diode_SMD:D_SOD-323
- D4: value 5V -> D_Schottky_Small
- J4: value PV Panel 1 -> PV Panel 2
- J5: value PV Panel 2 -> PV Panel 1
- L1: value 22uH -> 15uH; footprint Inductor_SMD:L_Bourns-SRN4018 -> Inductor_SMD:L_1210_3225Metric
- R1, R2: value 100k -> 47k
- R3: value 100k -> 10k
- R4: value 510R -> 330R
- R5: value 10k -> 100k
- R6: value 10k -> 31.2K
- U1: value ATSAMD21G18A -> STM32WL55CC; footprint Package_DFN_QFN:QFN-48-1EP_7x7mm_P0.5mm_EP5.3x5.3mm -> Package_DFN_QFN:QFN-48-1EP_7x7mm_P0.5mm_EP5.6x5.6mm
- U3: value INA226 -> TPS62152; footprint Package_SO:TSSOP-10_3x3mm_P0.5mm -> Package_DFN_QFN:VQFN-16-1EP_3x3mm_P0.5mm_EP1.68x1.68mm_ThermalVias
- moved R4 30.2 mm to (198.4, 82.5), turned to 0 degrees
- moved F1 28.6 mm to (198.9, 58.8), turned to 0 degrees
- moved L2 28.3 mm to (224.7, 78.6), turned to 270 degrees
- moved L1 23.7 mm to (195.6, 64.5), turned to 0 degrees
- moved J4 22.1 mm to (202.8, 84.6), turned to 0 degrees
- moved C2 19.8 mm to (199.3, 68.1)
- moved D2 19.3 mm to (196.2, 84.9), turned to 90 degrees
- moved C1 17.5 mm to (199.7, 63.8), turned to 180 degrees
- moved J5 16.4 mm to (210.6, 84.7), turned to 0 degrees
- moved C5 15.4 mm to (202.6, 61.3), turned to 180 degrees
- moved C8 14.3 mm to (215.1, 75.4), turned to 180 degrees
- moved R3 14.3 mm to (216.5, 73.9), turned to 0 degrees
- moved C7 13.3 mm to (215.2, 78.1), turned to 180 degrees
- moved R5 13.0 mm to (222.2, 74.3), turned to 90 degrees
- moved U3 12.1 mm to (219.3, 77.1), turned to 225 degrees
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- renumbered J8 to J2, J1 to J7
Connections:
- C1 pad 1: Net-(C1-Pad1) -> +3V3_EPS
- C2 pad 1: Net-(C2-Pad1) -> VDDSMPS-VDDRF
- C2 pad 2: GND -> Net-(C2-Pad2)
- C3 pad 1: /Power/VREF -> Net-(C2-Pad2)
- C3 pad 2: GND -> VDDRFF1-45
- C4 pad 1: Net-(C4-Pad1) -> +3V3_EPS
- C5 pad 1: +3V3_EPS -> Net-(C5-Pad1)
- C6 pad 1: +3V3_EPS -> VDDSMPS-VDDRF
- C7 pad 1: +3V3_EPS -> Net-(C7-Pad1)
- C8 pad 1: +3V3_EPS -> GND
- C8 pad 2: GND -> EPS_nRST
- C9 pad 1: +3V3_EPS -> PV
- D2 pad 1: /Power/ST1 -> GND
- D3 pad 1: GND -> PV
- D4 pad 1: Net-(C21-Pad1) -> PV
- D4 pad 2: GND -> Net-(D4-Pad2)
- J4 pad 2: Net-(D10-Pad2) -> Net-(D3-Pad2)
- J5 pad 2: Net-(D9-Pad2) -> Net-(D4-Pad2)
- L1 pad 1: PV -> Net-(L1-Pad1)
- L1 pad 2: Net-(L1-Pad2) -> VDDRFF1-45
- R1 pad 1: +3V3_SAT -> I2C_BUS_SDA
- R1 pad 2: SAT_nRST -> +3V3_EPS
- R2 pad 1: SAT_PWR_EN -> I2C_BUS_SCL
- R2 pad 2: GND -> +3V3_EPS
- R3 pad 1: +3V3_EPS -> GND
- R3 pad 2: EPS_nRST -> Net-(R3-Pad2)
- R4 pad 1: Net-(D1-Pad4) -> Net-(D2-Pad2)
- R4 pad 2: /RGB -> +3V3_EPS
- R5 pad 1: +3V3_EPS -> Net-(R5-Pad1)
- R5 pad 2: PWRMON_SCL -> +3V3_EPS
- R6 pad 1: +3V3_EPS -> Net-(R3-Pad2)
- R6 pad 2: PWRMON_SDA -> +3V3_EPS
- U1 pad 1: Net-(C1-Pad1) -> Net-(U1-Pad1)
- U1 pad 10: PWRMON_SCL -> Net-(U1-Pad10)
- U1 pad 11: /RGB -> +3V3_EPS
- U1 pad 12: OBC_OVTEMP -> Net-(U1-Pad12)
- U1 pad 13: I2C_BUS_SDA -> SPI_BUS_SCK
- U1 pad 14: I2C_BUS_SCL -> SPI_BUS_SDO
- U1 pad 15: SAT_PWR_EN -> SPI_BUS_SDI
- U1 pad 16: SAT_nRST -> Net-(U1-Pad16)
- U1 pad 17: +3V3_EPS -> I2C_BUS_SCL
- U1 pad 18: GND -> EPS_nRST
- U1 pad 19: SPI_BUS_SDI -> Net-(U1-Pad19)
- U1 pad 2: Net-(C2-Pad1) -> Net-(U1-Pad2)
- U1 pad 20: SPI_BUS_SCK -> Net-(U1-Pad20)
- U1 pad 21: SPI_BUS_SDO -> Net-(U1-Pad21)
- U1 pad 25: OBC_RX -> Net-(U1-Pad25)
- U1 pad 26: OBC_TX -> Net-(U1-Pad26)
- U1 pad 28: INT_IMU_OBC -> VDDSMPS-VDDRF
- U1 pad 29: /CS_FLASH -> VDDRFF1-45
- U1 pad 30: /SDI_FLASH -> Net-(U1-Pad30)
- U1 pad 31: /SDO_FLASH -> Net-(U1-Pad31)
- U1 pad 32: /SCK_FLASH -> Net-(U1-Pad32)
- U1 pad 33: USB_D- -> I2C_BUS_SDA
- U1 pad 34: USB_D+ -> Net-(U1-Pad34)
- U1 pad 35: GND -> Net-(U1-Pad35)
- U1 pad 36: +3V3_EPS -> Net-(U1-Pad36)
- U1 pad 37: Net-(U1-Pad37) -> +BATT
- U1 pad 40: EPS_nRST -> Net-(U1-Pad40)
- U1 pad 41: Net-(U1-Pad41) -> Net-(C5-Pad1)
- U1 pad 42: GND -> Net-(U1-Pad42)
- U1 pad 43: Net-(C4-Pad1) -> Net-(U1-Pad43)
- U1 pad 45: EPS_SWCLK -> VDDRFF1-45
- U1 pad 46: EPS_SWDIO -> VDDSMPS-VDDRF
- U1 pad 47: /5V_MEAS -> Net-(L1-Pad1)
- U1 pad 48: PWRMON_ALERT -> Net-(C2-Pad2)
- U1 pad 5: GND -> Net-(U1-Pad5)
- U1 pad 6: +3V3_EPS -> Net-(U1-Pad6)
- U1 pad 8: /3V3_MEAS -> Net-(U1-Pad8)
- U1 pad 9: PWRMON_SDA -> Net-(U1-Pad9)
- U3 pad 1: GND -> Net-(L2-Pad1)
- U3 pad 10: +BATT -> PV
- U3 pad 2: GND -> Net-(L2-Pad1)
- U3 pad 3: PWRMON_ALERT -> Net-(L2-Pad1)
- U3 pad 4: PWRMON_SDA -> Net-(R5-Pad1)
- U3 pad 5: PWRMON_SCL -> Net-(R3-Pad2)
- U3 pad 6: +BATT -> GND
- U3 pad 8: +BATT -> GND
- U3 pad 9: +BATT_MON -> Net-(C7-Pad1)
Routing:
- net SAT_PWR_EN: track 60.8 -> 0.15 mm, vias 6 -> 1
- net GND: track 55.8 -> 0.60 mm, vias 51 -> 8
- net +3V3_SAT: track 64.2 -> 27.0 mm, vias 9 -> 2
- net VBUS_JMP: track 36.7 -> 0.00 mm, vias 1 -> 0
- net +BATT_MON: track 35.6 -> 0.00 mm, vias 5 -> 0
- net /Power/VCHARGE: track 32.9 -> 0.00 mm, vias 5 -> 0
- net +5V_SAT: track 32.6 -> 1.38 mm, vias 4 -> 2
- net /Power/VOUT_PV: track 29.0 -> 0.00 mm, vias 3 -> 0
- net USB_D-: track 28.1 -> 0.00 mm, vias 3 -> 0
- net USB_D+: track 27.9 -> 0.00 mm, vias 2 -> 0
- net EPS_SWCLK: track 26.1 -> 0.00 mm, vias 1 -> 0
- net EPS_SWDIO: track 26.0 -> 0.00 mm, vias 1 -> 0
- net VDDSMPS-VDDRF: track 0.00 -> 25.3 mm, vias 0 -> 2
- net VDDRFF1-45: track 0.00 -> 24.2 mm, vias 0 -> 2
- net PWRMON_SCL: track 21.2 -> 0.00 mm, vias 2 -> 0
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- added copper zone on B.Cu, net +3V3_EPS
- added copper zone on In2.Cu, net GND
- removed copper zone on In2.Cu, net +3V3_EPS
- removed copper zone on B.Cu, net GND
Other:
- board text removed: "+"
- board text removed: "-"
- board text removed: "3V3"
- board text removed: "5V"
- board text removed: "A0"
- board text removed: "A1"
- board text removed: "A2"
- board text removed: "A3"
- board text removed: "A4"
- board text removed: "A5"
- board text removed: "AREF"
- board text removed: "BATT"
- board text removed: "BUS_SCK"
- board text removed: "BUS_SCL"
- board text removed: "BUS_SDA"
- board text removed: "BUS_SDI"
- board text removed: "BUS_SDO"
- board text removed: "CHG"
- board text removed: "D0"
- board text removed: "D1"
- board text removed: "D10"
- board text removed: "D2"
- board text removed: "D3"
- board text removed: "D30 - BUS_TX"
- board text removed: "D31 - BUS_RX"
- board text removed: "D32"
- board text removed: "D33"
- board text removed: "D4"
- board text removed: "D5"
- board text removed: "D6"
- board text removed: "D7"
- board text removed: "D8"
- board text removed: "D9"
- board text removed: "DynOSSAT-EDU"
- board text removed: "EPS v1.0"
- board text removed: "GND"
- board text removed: "OFF"
- board text removed: "ON"
- board text removed: "OVTEMP"
- board text removed: "PQBH-40 Bus"
- board text removed: "PV"
- board text removed: "PWR"
- board text removed: "SAT_PWR_EN"
- board text removed: "VBUS"
- board text removed: "~~"
